Commit message: wip: reformat urdf, large body

File: urdf/mimic_joint_gazebo_tutorial.urdf.xacro (robot description, xacro)
@@ -2,13 +2,59 @@
 <robot xmlns:xacro="http://ros.org/wiki/xacro"
   name="mimic_joint_gazebo_tutorial">
-  <xacro:macro name="box_inertial" params="x y z mass *origin">
+  <!-- - - - - - - - - - - Conventions - - - - - - - - - - -->
+  <!-- length is front to back (x-axis) -->
+  <!-- width goes left to right (y-axis) -->
+  <!-- height is up down (z-axis) -->
+  <!-- - - - - - - - - - - Parameters - - - - - - - - - - -->
+  <xacro:property name="bar_upper_limit" value="${pi/4}"/>
+  <xacro:property name="bar_lower_limit" value="0"/>
+  <xacro:property name="bar_effort" value="1000000"/>
+  <xacro:property name="bar_velocity" value="100"/>
+  <!-- - - - - - - - - - - Measurements - - - - - - - - - - -->
+  <!-- body -->
+  <xacro:property name="body_length" value="2"/>
+  <xacro:property name="body_width" value="3"/>
+  <xacro:property name="body_height" value="5"/>
+  <xacro:property name="body_mass" value="5"/>
+  <xacro:property name="bar_length" value="1"/>
+  <xacro:property name="bar_radius" value="0.1"/>
+  <xacro:property name="bar_mass" value="0.5"/>
+  <!-- - - - - - - - - - - Inertia Macros - - - - - - - - - - -->
+  <!-- Null -->
+  <xacro:macro name="null_inertial">
     <inertial>
-      <mass value="${mass}" />
-      <xacro:insert_block name="origin" />
-      <inertia ixx="${0.0833333 * mass * (y*y + z*z)}" ixy="0.0" ixz="0.0"
-        iyy="${0.0833333 * mass * (x*x + z*z)}" iyz="0.0"
-        izz="${0.0833333 * mass * (x*x + y*y)}" />
+      <mass value="0.001"/>
+      <inertia ixx="0.00001" ixy="0" ixz="0" iyy="0.00001" iyz="0" izz="0.00001"/>
     </inertial>
   </xacro:macro>
+  <!-- solid cuboid -->
+  <xacro:macro name="solid_cuboid_inertial"
+               params="length width height mass *origin">
+    <inertial>
+      <xacro:insert_block name="origin"/>
+      <mass value="${mass}"/>
+      <inertia ixx="${mass * (width * width + height * height) / 12}"
+               ixy="0" ixz="0"
+               iyy="${mass * (length * length + height * height) / 12}"
+               iyz="0"
+               izz="${mass * (length * length + width * width) / 12}"/>
+    </inertial>
+  </xacro:macro>
+  <!-- thick-walled cylindrical tube with open ends -->
+  <xacro:macro name="thick_walled_tube_inertial"
+               params="inner_rad outer_rad height mass">
+    <inertial>
+      <mass value="${mass}"/>
+      <inertia ixx="${(1 / 12) * mass * (3 * (inner_rad * inner_rad +
+                    outer_rad * outer_rad) + height * height)}"
+               ixy="0" ixz="0"
+               iyy="${(1 / 12) * mass * (3 * (inner_rad * inner_rad +
+                    outer_rad * outer_rad) + height * height)}"
+               iyz="0"
+               izz="${mass * (inner_rad * inner_rad +
+                    outer_rad * outer_rad) / 2}"/>
+    </inertial>
+  </xacro:macro>
+  <!-- - - - - - - - - - - colors - - - - - - - - - - -->
   <xacro:property name="material_yellow">
     <material name="yellow">
@@ -55,16 +101,12 @@
   </xacro:macro>
   <controller_plugin_gazebo />
-  <!-- base_footprint + base_link -->
-  <link name="base_footprint" />
-  <joint name="base_joint" type="fixed">
-    <origin xyz="0.0 0.0 0.025" />
-    <parent link="base_footprint" />
-    <child link="base_link" />
-  </joint>
-  <link name="base_link">
+  <!-- - - - - - - - - - - base_link - - - - - - - - - - -->
+  <link name="base_link" />
+  <!-- body-->
+  <link name="body">
     <visual>
       <origin xyz="0 0 0" />
       <geometry>
-        <box size="0.10 0.20 0.05" />
+        <box size="${body_length} ${body_width} ${body_height}" />
       </geometry>
       <xacro:insert_block name="material_yellow" />
@@ -73,18 +115,45 @@
       <origin xyz="0 0 0" />
       <geometry>
-        <box size="0.10 0.20 0.05" />
+        <box size="${body_length} ${body_width} ${body_height}" />
       </geometry>
     </collision>
-    <xacro:box_inertial mass="1.0" x="0.10" y="0.20" z="0.05">
-      <origin xyz="0 0 0" />
-    </xacro:box_inertial>
+    <xacro:solid_cuboid_inertial
+        length="${body_length}" width="${body_width}"
+        height="${body_height}" mass="${body_mass}">
+      <origin xyz="0 0 0"/>
+    </xacro:solid_cuboid_inertial>
   </link>
-  <gazebo reference="base_link">
+  <joint name="body_to_base" type="fixed">
+    <origin xyz="0.0 0.0 0.0" />
+    <parent link="base_link" />
+    <child link="body" />
+  </joint>
+  <gazebo reference="body">
     <material>Gazebo/Yellow</material>
   </gazebo>
   <!-- right finger -->
+  <link name="right_finger">
+    <visual>
+      <origin xyz="0 0.10 0" />
+      <geometry>
+        <box size="0.02 0.20 0.02" />
+      </geometry>
+      <xacro:insert_block name="material_green" />
+    </visual>
+    <collision>
+      <origin xyz="0 0.10 0" />
+      <geometry>
+        <box size="0.02 0.20 0.02" />
+      </geometry>
+    </collision>
+    <xacro:solid_cuboid_inertial
+        length="${0.02}" width="${0.20}"
+        height="${0.02}" mass="${0.1}">
+      <origin xyz="0 0 0"/>
+    </xacro:solid_cuboid_inertial>
+  </link>
   <joint name="right_finger_joint" type="revolute">
     <origin xyz="0.0 -0.10 0.0" rpy="0 0 ${pi}" />
-    <parent link="base_link" />
+    <parent link="body" />
     <child link="right_finger" />
     <axis xyz="1 0 0" />
@@ -92,22 +161,4 @@
     <dynamics damping="0.02" friction="0.0" />
   </joint>
-  <link name="right_finger">
-    <visual>
-      <origin xyz="0 0.10 0" />
-      <geometry>
-        <box size="0.02 0.20 0.02" />
-      </geometry>
-      <xacro:insert_block name="material_green" />
-    </visual>
-    <collision>
-      <origin xyz="0 0.10 0" />
-      <geometry>
-        <box size="0.02 0.20 0.02" />
-      </geometry>
-    </collision>
-    <xacro:box_inertial mass="0.1" x="0.02" y="0.20" z="0.02">
-      <origin xyz="0 0.10 0" />
-    </xacro:box_inertial>
-  </link>
   <gazebo reference="right_finger">
     <material>Gazebo/Green</material>
@@ -125,5 +176,5 @@
   <joint name="left_finger_joint" type="revolute">
     <origin xyz="0.0 0.10 0.0" />
-    <parent link="base_link" />
+    <parent link="body" />
     <child link="left_finger" />
     <axis xyz="1 0 0" />
@@ -149,7 +200,9 @@
       </geometry>
     </collision>
-    <xacro:box_inertial mass="0.1" x="0.02" y="0.20" z="0.02">
-      <origin xyz="0 0.10 0" />
-    </xacro:box_inertial>
+    <xacro:solid_cuboid_inertial
+        length="${0.02}" width="${0.20}"
+        height="${0.02}" mass="${0.1}">
+      <origin xyz="0 0 0"/>
+    </xacro:solid_cuboid_inertial>
   </link>
   <gazebo reference="left_finger">

Commit message: wip: reorg urdf, change location of fingers

File: urdf/mimic_joint_gazebo_tutorial.urdf.xacro (robot description, xacro)
@@ -135,5 +135,4 @@
   <link name="right_finger">
     <visual>
-      <origin xyz="0 0.10 0" />
       <geometry>
         <box size="0.02 0.20 0.02" />
@@ -142,5 +141,4 @@
     </visual>
     <collision>
-      <origin xyz="0 0.10 0" />
       <geometry>
         <box size="0.02 0.20 0.02" />
@@ -154,5 +152,5 @@
   </link>
   <joint name="right_finger_joint" type="revolute">
-    <origin xyz="0.0 -0.10 0.0" rpy="0 0 ${pi}" />
+    <origin xyz="0.0 -0.10 ${body_height/2}" rpy="0 0 ${pi}" />
     <parent link="body" />
     <child link="right_finger" />
@@ -161,7 +159,4 @@
     <dynamics damping="0.02" friction="0.0" />
   </joint>
-  <gazebo reference="right_finger">
-    <material>Gazebo/Green</material>
-  </gazebo>
   <transmission name="right_finger_joint_trans">
     <type>transmission_interface/SimpleTransmission</type>
@@ -173,7 +168,28 @@
     </actuator>
   </transmission>
+  <gazebo reference="right_finger">
+    <material>Gazebo/Green</material>
+  </gazebo>
   <!-- left finger -->
+  <link name="left_finger">
+    <visual>
+      <geometry>
+        <box size="0.02 0.20 0.02" />
+      </geometry>
+      <xacro:insert_block name="material_red" />
+    </visual>
+    <collision>
+      <geometry>
+        <box size="0.02 0.20 0.02" />
+      </geometry>
+    </collision>
+    <xacro:solid_cuboid_inertial
+        length="${0.02}" width="${0.20}"
+        height="${0.02}" mass="${0.1}">
+      <origin xyz="0 0 0"/>
+    </xacro:solid_cuboid_inertial>
+  </link>
   <joint name="left_finger_joint" type="revolute">
-    <origin xyz="0.0 0.10 0.0" />
+    <origin xyz="0.0 0.10 ${body_height/2}" />
     <parent link="body" />
     <child link="left_finger" />
@@ -183,30 +199,10 @@
     <dynamics damping="0.02" friction="0.0" />
   </joint>
+  <gazebo reference="left_finger">
+    <material>Gazebo/Red</material>
+  </gazebo>
   <xacro:mimic_joint_plugin_gazebo name_prefix="left_finger_joint"
     parent_joint="right_finger_joint" mimic_joint="left_finger_joint"
     has_pid="true" multiplier="1.0" max_effort="10.0" />
-  <link name="left_finger">
-    <visual>
-      <origin xyz="0 0.10 0" />
-      <geometry>
-        <box size="0.02 0.20 0.02" />
-      </geometry>
-      <xacro:insert_block name="material_red" />
-    </visual>
-    <collision>
-      <origin xyz="0 0.10 0" />
-      <geometry>
-        <box size="0.02 0.20 0.02" />
-      </geometry>
-    </collision>
-    <xacro:solid_cuboid_inertial
-        length="${0.02}" width="${0.20}"
-        height="${0.02}" mass="${0.1}">
-      <origin xyz="0 0 0"/>
-    </xacro:solid_cuboid_inertial>
-  </link>
-  <gazebo reference="left_finger">
-    <material>Gazebo/Red</material>
-  </gazebo>
   <!-- DO NOT add a transmission for the left finger joint. We want the left
        finger joint to be controlled by the mimic plugin. If we add a

Commit message: wip: larger figner and cylinder, next xacro macro

File: urdf/mimic_joint_gazebo_tutorial.urdf.xacro (robot description, xacro)
@@ -136,5 +136,5 @@
     <visual>
       <geometry>
-        <box size="0.02 0.20 0.02" />
+        <cylinder length="${bar_length}" radius="${bar_radius}"/>
       </geometry>
       <xacro:insert_block name="material_green" />
@@ -142,15 +142,13 @@
     <collision>
       <geometry>
-        <box size="0.02 0.20 0.02" />
+        <cylinder length="${bar_length}" radius="${bar_radius}"/>
       </geometry>
     </collision>
-    <xacro:solid_cuboid_inertial
-        length="${0.02}" width="${0.20}"
-        height="${0.02}" mass="${0.1}">
-      <origin xyz="0 0 0"/>
-    </xacro:solid_cuboid_inertial>
+    <xacro:thick_walled_tube_inertial
+      inner_rad="0.0" outer_rad="${bar_radius}"
+      height="${bar_length}" mass="${bar_mass}"/>
   </link>
   <joint name="right_finger_joint" type="revolute">
-    <origin xyz="0.0 -0.10 ${body_height/2}" rpy="0 0 ${pi}" />
+    <origin xyz="0.0 ${bar_length/2} ${body_height/2+bar_length/2}" rpy="0 0 ${pi}" />
     <parent link="body" />
     <child link="right_finger" />

Commit message: wip: bars stick straight out and move down, next I need to add tips with sensors and mimic the sensor joints

File: urdf/mimic_joint_gazebo_tutorial.urdf.xacro (robot description, xacro)
@@ -6,4 +6,11 @@
   <!-- width goes left to right (y-axis) -->
   <!-- height is up down (z-axis) -->
+  <!-- reflection convention -->
+  <!--
+  front +1
+  back  -1
+  left  +1
+  right -1
+  -->
   <!-- - - - - - - - - - - Parameters - - - - - - - - - - -->
   <xacro:property name="bar_upper_limit" value="${pi/4}"/>
@@ -132,88 +139,50 @@
     <material>Gazebo/Yellow</material>
   </gazebo>
-  <!-- right finger -->
-  <link name="right_finger">
-    <visual>
-      <geometry>
-        <cylinder length="${bar_length}" radius="${bar_radius}"/>
-      </geometry>
-      <xacro:insert_block name="material_green" />
-    </visual>
-    <collision>
-      <geometry>
-        <cylinder length="${bar_length}" radius="${bar_radius}"/>
-      </geometry>
-    </collision>
-    <xacro:thick_walled_tube_inertial
-      inner_rad="0.0" outer_rad="${bar_radius}"
-      height="${bar_length}" mass="${bar_mass}"/>
-  </link>
-  <joint name="right_finger_joint" type="revolute">
-    <origin xyz="0.0 ${bar_length/2} ${body_height/2+bar_length/2}" rpy="0 0 ${pi}" />
-    <parent link="body" />
-    <child link="right_finger" />
-    <axis xyz="1 0 0" />
-    <limit lower="0" upper="${pi / 2}" velocity="0.7" effort="1000" />
-    <dynamics damping="0.02" friction="0.0" />
-  </joint>
-  <transmission name="right_finger_joint_trans">
+  <!-- bars -->
+  <xacro:macro name="bar" params="lr_prefix lr_reflect">
+    <link name="${lr_prefix}_bar">
+      <visual>
+        <origin xyz="0 0 ${bar_length/2}"/>
+        <geometry>
+          <cylinder length="${bar_length}" radius="${bar_radius}"/>
+        </geometry>
+      </visual>
+      <collision>
+        <geometry>
+          <cylinder length="${bar_length}" radius="${bar_radius}"/>
+        </geometry>
+      </collision>
+      <xacro:thick_walled_tube_inertial
+        inner_rad="0.0" outer_rad="${bar_radius}"
+        height="${bar_length}" mass="${bar_mass}"/>
+    </link>
+    <joint name="${lr_prefix}_joint" type="revolute">
+      <origin xyz="${body_length/2} ${lr_reflect*body_width/4} 0.0" rpy="0 ${pi/2} 0" />
+      <parent link="body" />
+      <child link="${lr_prefix}_bar" />
+      <axis xyz="0 1 0" />
+      <limit lower="0" upper="${pi / 2}" velocity="0.7" effort="1000" />
+      <dynamics damping="0.02" friction="0.0" />
+    </joint>
+  </xacro:macro>
+  <xacro:bar lr_prefix="right" lr_reflect="-1"/>
+  <transmission name="right_trans">
     <type>transmission_interface/SimpleTransmission</type>
-    <joint name="right_finger_joint">
+    <joint name="right_joint">
       <hardwareInterface>hardware_interface/PositionJointInterface</hardwareInterface>
     </joint>
-    <actuator name="right_finger_joint_motor">
+    <actuator name="right_motor">
       <mechanicalReduction>1</mechanicalReduction>
     </actuator>
   </transmission>
-  <gazebo reference="right_finger">
+  <xacro:bar lr_prefix="left" lr_reflect="1"/>
+  <gazebo reference="right_bar">
     <material>Gazebo/Green</material>
   </gazebo>
-  <!-- left finger -->
-  <link name="left_finger">
-    <visual>
-      <geometry>
-        <box size="0.02 0.20 0.02" />
-      </geometry>
-      <xacro:insert_block name="material_red" />
-    </visual>
-    <collision>
-      <geometry>
-        <box size="0.02 0.20 0.02" />
-      </geometry>
-    </collision>
-    <xacro:solid_cuboid_inertial
-        length="${0.02}" width="${0.20}"
-        height="${0.02}" mass="${0.1}">
-      <origin xyz="0 0 0"/>
-    </xacro:solid_cuboid_inertial>
-  </link>
-  <joint name="left_finger_joint" type="revolute">
-    <origin xyz="0.0 0.10 ${body_height/2}" />
-    <parent link="body" />
-    <child link="left_finger" />
-    <axis xyz="1 0 0" />
-    <limit lower="0" upper="${pi / 2}" velocity="0.7" effort="1000" />
-    <mimic joint="right_finger_joint" multiplier="1" offset="0" />
-    <dynamics damping="0.02" friction="0.0" />
-  </joint>
   <gazebo reference="left_finger">
     <material>Gazebo/Red</material>
   </gazebo>
-  <xacro:mimic_joint_plugin_gazebo name_prefix="left_finger_joint"
-    parent_joint="right_finger_joint" mimic_joint="left_finger_joint"
+  <xacro:mimic_joint_plugin_gazebo name_prefix="left_joint"
+    parent_joint="right_joint" mimic_joint="left_joint"
     has_pid="true" multiplier="1.0" max_effort="10.0" />
-  <!-- DO NOT add a transmission for the left finger joint. We want the left
-       finger joint to be controlled by the mimic plugin. If we add a
-       transmission, the ros_control plugin will try to control this joint. -->
-  <!--
-  <transmission name="left_finger_joint_trans">
-    <type>transmission_interface/SimpleTransmission</type>
-    <joint name="left_finger_joint">
-      <hardwareInterface>hardware_interface/PositionJointInterface</hardwareInterface>
-    </joint>
-    <actuator name="left_finger_joint_motor">
-      <mechanicalReduction>1</mechanicalReduction>
-    </actuator>
-  </transmission>
-  -->
 </robot>

Commit message: wip: tip on end of bar

File: urdf/mimic_joint_gazebo_tutorial.urdf.xacro (robot description, xacro)
@@ -139,5 +139,5 @@
     <material>Gazebo/Yellow</material>
   </gazebo>
-  <!-- bars -->
+  <!-- bar macro -->
   <xacro:macro name="bar" params="lr_prefix lr_reflect">
     <link name="${lr_prefix}_bar">
@@ -166,4 +166,5 @@
     </joint>
   </xacro:macro>
+  <!-- right bar -->
   <xacro:bar lr_prefix="right" lr_reflect="-1"/>
   <transmission name="right_trans">
@@ -176,13 +177,67 @@
     </actuator>
   </transmission>
-  <xacro:bar lr_prefix="left" lr_reflect="1"/>
   <gazebo reference="right_bar">
     <material>Gazebo/Green</material>
   </gazebo>
+<!-- tip sensor -->
+<link name="tip">
+  <visual>
+    <origin xyz="0 0 0" rpy="0 0 0"/>
+    <geometry>
+      <sphere radius="0.01"/>
+    </geometry>
+    <xacro:insert_block name="material_yellow" />
+  </visual>
+  <xacro:null_inertial/>
+</link>
+<joint name="tip_to_bar" type="fixed">
+  <parent link="right_bar"/>
+  <child link="tip"/>
+  <origin xyz="0 0 ${body_length/2}" rpy="0 0 0"/>
+</joint>
+<gazebo reference="tip">
+   <sensor type="ray" name="tip_sensor">
+      <alwaysOn>true</alwaysOn>
+      <update_rate>50</update_rate>
+      <visualize>true</visualize>
+      <topic>/tip_sensor/height_above_ground</topic>
+      <ray>
+         <scan>
+            <horizontal>
+               <samples>1</samples>
+               <resolution>1.0</resolution>
+               <min_angle>-0.01</min_angle>
+               <max_angle>0.01</max_angle>
+            </horizontal>
+            <vertical>
+               <samples>1</samples>
+               <resolution>1</resolution>
+               <min_angle>-0.01</min_angle>
+               <max_angle>0.01</max_angle>
+            </vertical>
+         </scan>
+         <range>
+            <min>0.01</min>
+            <max>3.75</max>
+            <resolution>0.02</resolution>
+         </range>
+      </ray>
+      <plugin filename="libgazebo_ros_range.so" name="gazebo_ros_range">
+         <gaussianNoise>0.005</gaussianNoise>
+         <updateRate>5</updateRate>
+         <topicName>/radar_sim/height_above_ground</topicName>
+         <frameName>radar_panel_tip</frameName>
+         <radiation>infrared</radiation>
+         <fov>0.02</fov>
+      </plugin>
+   </sensor>
+</gazebo>
+  <!-- left bar -->
+  <xacro:bar lr_prefix="left" lr_reflect="1"/>
+  <xacro:mimic_joint_plugin_gazebo name_prefix="left_joint"
+    parent_joint="right_joint" mimic_joint="left_joint"
+    has_pid="true" multiplier="1.0" max_effort="10.0" />
   <gazebo reference="left_finger">
     <material>Gazebo/Red</material>
   </gazebo>
-  <xacro:mimic_joint_plugin_gazebo name_prefix="left_joint"
-    parent_joint="right_joint" mimic_joint="left_joint"
-    has_pid="true" multiplier="1.0" max_effort="10.0" />
 </robot>

Commit message: wip:trying to figure out why everything blows up

File: urdf/mimic_joint_gazebo_tutorial.urdf.xacro (robot description, xacro)
@@ -23,5 +23,5 @@
   <xacro:property name="body_width" value="3"/>
   <xacro:property name="body_height" value="5"/>
-  <xacro:property name="body_mass" value="5"/>
+  <xacro:property name="body_mass" value="500"/>
   <xacro:property name="bar_length" value="1"/>
   <xacro:property name="bar_radius" value="0.1"/>
@@ -31,5 +31,5 @@
   <xacro:macro name="null_inertial">
     <inertial>
-      <mass value="0.001"/>
+      <mass value="0.0001"/>
       <inertia ixx="0.00001" ixy="0" ixz="0" iyy="0.00001" iyz="0" izz="0.00001"/>
     </inertial>
@@ -162,6 +162,6 @@
       <child link="${lr_prefix}_bar" />
       <axis xyz="0 1 0" />
-      <limit lower="0" upper="${pi / 2}" velocity="0.7" effort="1000" />
-      <dynamics damping="0.02" friction="0.0" />
+      <limit lower="0" upper="${pi / 2}" velocity="0.7" effort="10" />
+      <dynamics damping="0.02" friction="0.1" />
     </joint>
   </xacro:macro>
@@ -181,5 +181,5 @@
   </gazebo>
 <!-- tip sensor -->
-<link name="tip">
+<!-- <link name="tip">
   <visual>
     <origin xyz="0 0 0" rpy="0 0 0"/>
@@ -191,13 +191,17 @@
   <xacro:null_inertial/>
 </link>
-<joint name="tip_to_bar" type="fixed">
+<joint name="tip_to_bar" type="revolute">
   <parent link="right_bar"/>
   <child link="tip"/>
   <origin xyz="0 0 ${body_length/2}" rpy="0 0 0"/>
+  <axis xyz="0 1 0" />
+  <limit lower="0" upper="${pi / 2}" velocity="0.7" effort="1" />
+  <mimic joint="right_joint" multiplier="-1" offset="0" />
+  <dynamics damping="0.2" friction="0.1" />
 </joint>
 <gazebo reference="tip">
    <sensor type="ray" name="tip_sensor">
       <alwaysOn>true</alwaysOn>
-      <update_rate>50</update_rate>
+      <update_rate>30</update_rate>
       <visualize>true</visualize>
       <topic>/tip_sensor/height_above_ground</topic>
@@ -226,18 +230,18 @@
          <gaussianNoise>0.005</gaussianNoise>
          <updateRate>5</updateRate>
-         <topicName>/radar_sim/height_above_ground</topicName>
-         <frameName>radar_panel_tip</frameName>
+         <topicName>/tip_sensor/height_above_ground</topicName>
+         <frameName>tip</frameName>
          <radiation>infrared</radiation>
          <fov>0.02</fov>
       </plugin>
    </sensor>
-</gazebo>
+</gazebo> -->
   <!-- left bar -->
   <xacro:bar lr_prefix="left" lr_reflect="1"/>
-  <xacro:mimic_joint_plugin_gazebo name_prefix="left_joint"
-    parent_joint="right_joint" mimic_joint="left_joint"
-    has_pid="true" multiplier="1.0" max_effort="10.0" />
   <gazebo reference="left_finger">
     <material>Gazebo/Red</material>
   </gazebo>
+  <xacro:mimic_joint_plugin_gazebo name_prefix="mimic_joint"
+    parent_joint="right_joint" mimic_joint="left_joint"
+    has_pid="true" multiplier="1.0" max_effort="1" />
 </robot>
