Commit message: wip: almost there

File: urdf/mimic_joint_gazebo_tutorial.urdf.xacro (robot description, xacro)
@@ -162,16 +162,13 @@
       <child link="${lr_prefix}_bar" />
       <axis xyz="0 1 0" />
-      <limit lower="0" upper="${pi / 2}" velocity="0.7" effort="10" />
+      <limit lower="0" upper="${pi / 2}" velocity="0.7" effort="1000" />
       <dynamics damping="0.02" friction="0.1" />
     </joint>
-  </xacro:macro>
-  <!-- right bar -->
-  <xacro:bar lr_prefix="right" lr_reflect="-1"/>
-  <transmission name="right_trans">
+    <transmission name="${lr_prefix}_trans">
     <type>transmission_interface/SimpleTransmission</type>
-    <joint name="right_joint">
+    <joint name="${lr_prefix}_joint">
       <hardwareInterface>hardware_interface/PositionJointInterface</hardwareInterface>
     </joint>
-    <actuator name="right_motor">
+    <actuator name="${lr_prefix}_motor">
       <mechanicalReduction>1</mechanicalReduction>
     </actuator>
@@ -180,6 +177,9 @@
     <material>Gazebo/Green</material>
   </gazebo>
+  </xacro:macro>
+  <!-- right bar -->
+  <xacro:bar lr_prefix="right" lr_reflect="-1"/>
 <!-- tip sensor -->
-<!-- <link name="tip">
+<link name="tip">
   <visual>
     <origin xyz="0 0 0" rpy="0 0 0"/>
@@ -192,15 +192,14 @@
 </link>
 <joint name="tip_to_bar" type="revolute">
-  <parent link="right_bar"/>
+  <parent link="left_bar"/>
   <child link="tip"/>
   <origin xyz="0 0 ${body_length/2}" rpy="0 0 0"/>
   <axis xyz="0 1 0" />
-  <limit lower="0" upper="${pi / 2}" velocity="0.7" effort="1" />
-  <mimic joint="right_joint" multiplier="-1" offset="0" />
+  <limit lower="${-pi}" upper="${pi}" velocity="0.35" effort="1" />
+  <mimic joint="right_joint" multiplier="1" offset="0" />
   <dynamics damping="0.2" friction="0.1" />
 </joint>
 <gazebo reference="tip">
    <sensor type="ray" name="tip_sensor">
-      <alwaysOn>true</alwaysOn>
       <update_rate>30</update_rate>
       <visualize>true</visualize>
@@ -236,12 +235,12 @@
       </plugin>
    </sensor>
-</gazebo> -->
+</gazebo>
   <!-- left bar -->
   <xacro:bar lr_prefix="left" lr_reflect="1"/>
-  <gazebo reference="left_finger">
+  <gazebo reference="left_bar">
     <material>Gazebo/Red</material>
   </gazebo>
   <xacro:mimic_joint_plugin_gazebo name_prefix="mimic_joint"
-    parent_joint="right_joint" mimic_joint="left_joint"
-    has_pid="true" multiplier="1.0" max_effort="1" />
+    parent_joint="right_joint" mimic_joint="tip_to_bar"
+    has_pid="false" multiplier="${-1.0}" max_effort="1" />
 </robot>

Commit message: wip: right tip sensor mimics the right bar, need to clean up and duplicate on left

File: urdf/mimic_joint_gazebo_tutorial.urdf.xacro (robot description, xacro)
@@ -192,5 +192,5 @@
 </link>
 <joint name="tip_to_bar" type="revolute">
-  <parent link="left_bar"/>
+  <parent link="right_bar"/>
   <child link="tip"/>
   <origin xyz="0 0 ${body_length/2}" rpy="0 0 0"/>

Commit message: wip: reorg for clarity

File: urdf/mimic_joint_gazebo_tutorial.urdf.xacro (robot description, xacro)
@@ -79,4 +79,5 @@
     </material>
   </xacro:property>
+  <!-- - - - - - - - - - - gazebo plugins - - - - - - - - - - -->
   <xacro:macro name="mimic_joint_plugin_gazebo" params="name_prefix parent_joint mimic_joint has_pid:=false multiplier:=1.0 offset:=0 sensitiveness:=0.0 max_effort:=1.0 robot_namespace:=''">
     <gazebo>
@@ -97,4 +98,7 @@
     </gazebo>
   </xacro:macro>
+  <xacro:mimic_joint_plugin_gazebo name_prefix="mimic_joint"
+    parent_joint="right_joint" mimic_joint="tip_to_bar"
+    has_pid="false" multiplier="${-1.0}" max_effort="1" />
   <xacro:macro name="controller_plugin_gazebo" params="robot_namespace:=''">
     <gazebo>
@@ -108,4 +112,10 @@
   </xacro:macro>
   <controller_plugin_gazebo />
+  <gazebo reference="right_bar">
+    <material>Gazebo/Green</material>
+  </gazebo>
+  <gazebo reference="left_bar">
+    <material>Gazebo/Red</material>
+  </gazebo>
   <!-- - - - - - - - - - - base_link - - - - - - - - - - -->
   <link name="base_link" />
@@ -166,81 +176,72 @@
     </joint>
     <transmission name="${lr_prefix}_trans">
-    <type>transmission_interface/SimpleTransmission</type>
-    <joint name="${lr_prefix}_joint">
-      <hardwareInterface>hardware_interface/PositionJointInterface</hardwareInterface>
-    </joint>
-    <actuator name="${lr_prefix}_motor">
-      <mechanicalReduction>1</mechanicalReduction>
-    </actuator>
-  </transmission>
-  <gazebo reference="right_bar">
-    <material>Gazebo/Green</material>
-  </gazebo>
+      <type>transmission_interface/SimpleTransmission</type>
+      <joint name="${lr_prefix}_joint">
+        <hardwareInterface>hardware_interface/PositionJointInterface</hardwareInterface>
+      </joint>
+      <actuator name="${lr_prefix}_motor">
+        <mechanicalReduction>1</mechanicalReduction>
+      </actuator>
+    </transmission>
   </xacro:macro>
   <!-- right bar -->
   <xacro:bar lr_prefix="right" lr_reflect="-1"/>
-<!-- tip sensor -->
-<link name="tip">
-  <visual>
-    <origin xyz="0 0 0" rpy="0 0 0"/>
-    <geometry>
-      <sphere radius="0.01"/>
-    </geometry>
-    <xacro:insert_block name="material_yellow" />
-  </visual>
-  <xacro:null_inertial/>
-</link>
-<joint name="tip_to_bar" type="revolute">
-  <parent link="right_bar"/>
-  <child link="tip"/>
-  <origin xyz="0 0 ${body_length/2}" rpy="0 0 0"/>
-  <axis xyz="0 1 0" />
-  <limit lower="${-pi}" upper="${pi}" velocity="0.35" effort="1" />
-  <mimic joint="right_joint" multiplier="1" offset="0" />
-  <dynamics damping="0.2" friction="0.1" />
-</joint>
-<gazebo reference="tip">
-   <sensor type="ray" name="tip_sensor">
-      <update_rate>30</update_rate>
-      <visualize>true</visualize>
-      <topic>/tip_sensor/height_above_ground</topic>
-      <ray>
-         <scan>
-            <horizontal>
-               <samples>1</samples>
-               <resolution>1.0</resolution>
-               <min_angle>-0.01</min_angle>
-               <max_angle>0.01</max_angle>
-            </horizontal>
-            <vertical>
-               <samples>1</samples>
-               <resolution>1</resolution>
-               <min_angle>-0.01</min_angle>
-               <max_angle>0.01</max_angle>
-            </vertical>
-         </scan>
-         <range>
-            <min>0.01</min>
-            <max>3.75</max>
-            <resolution>0.02</resolution>
-         </range>
-      </ray>
-      <plugin filename="libgazebo_ros_range.so" name="gazebo_ros_range">
-         <gaussianNoise>0.005</gaussianNoise>
-         <updateRate>5</updateRate>
-         <topicName>/tip_sensor/height_above_ground</topicName>
-         <frameName>tip</frameName>
-         <radiation>infrared</radiation>
-         <fov>0.02</fov>
-      </plugin>
-   </sensor>
-</gazebo>
   <!-- left bar -->
   <xacro:bar lr_prefix="left" lr_reflect="1"/>
-  <gazebo reference="left_bar">
-    <material>Gazebo/Red</material>
-  </gazebo>
-  <xacro:mimic_joint_plugin_gazebo name_prefix="mimic_joint"
-    parent_joint="right_joint" mimic_joint="tip_to_bar"
-    has_pid="false" multiplier="${-1.0}" max_effort="1" />
+  <!-- tip sensor -->
+  <link name="tip">
+    <visual>
+      <origin xyz="0 0 0" rpy="0 0 0"/>
+      <geometry>
+        <sphere radius="0.01"/>
+      </geometry>
+      <xacro:insert_block name="material_yellow" />
+    </visual>
+    <xacro:null_inertial/>
+  </link>
+  <joint name="tip_to_bar" type="revolute">
+    <parent link="right_bar"/>
+    <child link="tip"/>
+    <origin xyz="0 0 ${body_length/2}" rpy="0 0 0"/>
+    <axis xyz="0 1 0" />
+    <limit lower="${-pi}" upper="${pi}" velocity="0.35" effort="1" />
+    <mimic joint="right_joint" multiplier="1" offset="0" />
+    <dynamics damping="0.2" friction="0.1" />
+  </joint>
+  <gazebo reference="tip">
+    <sensor type="ray" name="tip_sensor">
+        <update_rate>30</update_rate>
+        <visualize>true</visualize>
+        <topic>/tip_sensor/height_above_ground</topic>
+        <ray>
+          <scan>
+              <horizontal>
+                <samples>1</samples>
+                <resolution>1.0</resolution>
+                <min_angle>-0.01</min_angle>
+                <max_angle>0.01</max_angle>
+              </horizontal>
+              <vertical>
+                <samples>1</samples>
+                <resolution>1</resolution>
+                <min_angle>-0.01</min_angle>
+                <max_angle>0.01</max_angle>
+              </vertical>
+          </scan>
+          <range>
+              <min>0.01</min>
+              <max>3.75</max>
+              <resolution>0.02</resolution>
+          </range>
+        </ray>
+      <plugin filename="libgazebo_ros_range.so" name="gazebo_ros_range">
+        <gaussianNoise>0.005</gaussianNoise>
+        <updateRate>5</updateRate>
+        <topicName>/tip_sensor/height_above_ground</topicName>
+        <frameName>tip</frameName>
+        <radiation>infrared</radiation>
+        <fov>0.02</fov>
+      </plugin>
+    </sensor>
+  </gazebo>
 </robot>

Commit message: wip: using macros for tip and tip sensor

File: urdf/mimic_joint_gazebo_tutorial.urdf.xacro (robot description, xacro)
@@ -99,5 +99,5 @@
   </xacro:macro>
   <xacro:mimic_joint_plugin_gazebo name_prefix="mimic_joint"
-    parent_joint="right_joint" mimic_joint="tip_to_bar"
+    parent_joint="right_joint" mimic_joint="right_tip_joint"
     has_pid="false" multiplier="${-1.0}" max_effort="1" />
   <xacro:macro name="controller_plugin_gazebo" params="robot_namespace:=''">
@@ -185,63 +185,69 @@
     </transmission>
   </xacro:macro>
+  <!-- tip sensor -->
+  <xacro:macro name="tip" params="lr_prefix">
+    <link name="${lr_prefix}_tip">
+      <visual>
+        <origin xyz="0 0 0" rpy="0 0 0"/>
+        <geometry>
+          <sphere radius="0.01"/>
+        </geometry>
+        <xacro:insert_block name="material_yellow" />
+      </visual>
+      <xacro:null_inertial/>
+    </link>
+    <joint name="${lr_prefix}_tip_joint" type="revolute">
+      <parent link="${lr_prefix}_bar"/>
+      <child link="${lr_prefix}_tip"/>
+      <origin xyz="0 0 ${body_length/2}" rpy="0 0 0"/>
+      <axis xyz="0 1 0" />
+      <limit lower="${-pi}" upper="${pi}" velocity="0.35" effort="1" />
+      <mimic joint="${lr_prefix}_joint" multiplier="1" offset="0" />
+      <dynamics damping="0.2" friction="0.1" />
+    </joint>
+  </xacro:macro>
+  <xacro:macro name="tip_sensor" params="lr_prefix">
+    <gazebo reference="${lr_prefix}_tip">
+      <sensor type="ray" name="${lr_prefix}_tip_sensor">
+          <update_rate>30</update_rate>
+          <visualize>true</visualize>
+          <topic>/${lr_prefix}_tip_sensor/height_above_ground</topic>
+          <ray>
+            <scan>
+                <horizontal>
+                  <samples>1</samples>
+                  <resolution>1.0</resolution>
+                  <min_angle>-0.01</min_angle>
+                  <max_angle>0.01</max_angle>
+                </horizontal>
+                <vertical>
+                  <samples>1</samples>
+                  <resolution>1</resolution>
+                  <min_angle>-0.01</min_angle>
+                  <max_angle>0.01</max_angle>
+                </vertical>
+            </scan>
+            <range>
+                <min>0.01</min>
+                <max>3.75</max>
+                <resolution>0.02</resolution>
+            </range>
+          </ray>
+        <plugin filename="libgazebo_ros_range.so" name="gazebo_ros_range">
+          <gaussianNoise>0.005</gaussianNoise>
+          <updateRate>5</updateRate>
+          <topicName>/${lr_prefix}_tip_sensor/height_above_ground</topicName>
+          <frameName>${lr_prefix}_tip</frameName>
+          <radiation>infrared</radiation>
+          <fov>0.02</fov>
+        </plugin>
+      </sensor>
+    </gazebo>
+  </xacro:macro>
   <!-- right bar -->
   <xacro:bar lr_prefix="right" lr_reflect="-1"/>
+  <xacro:tip lr_prefix="right"/>
+  <xacro:tip_sensor lr_prefix="right"/>
   <!-- left bar -->
   <xacro:bar lr_prefix="left" lr_reflect="1"/>
-  <!-- tip sensor -->
-  <link name="tip">
-    <visual>
-      <origin xyz="0 0 0" rpy="0 0 0"/>
-      <geometry>
-        <sphere radius="0.01"/>
-      </geometry>
-      <xacro:insert_block name="material_yellow" />
-    </visual>
-    <xacro:null_inertial/>
-  </link>
-  <joint name="tip_to_bar" type="revolute">
-    <parent link="right_bar"/>
-    <child link="tip"/>
-    <origin xyz="0 0 ${body_length/2}" rpy="0 0 0"/>
-    <axis xyz="0 1 0" />
-    <limit lower="${-pi}" upper="${pi}" velocity="0.35" effort="1" />
-    <mimic joint="right_joint" multiplier="1" offset="0" />
-    <dynamics damping="0.2" friction="0.1" />
-  </joint>
-  <gazebo reference="tip">
-    <sensor type="ray" name="tip_sensor">
-        <update_rate>30</update_rate>
-        <visualize>true</visualize>
-        <topic>/tip_sensor/height_above_ground</topic>
-        <ray>
-          <scan>
-              <horizontal>
-                <samples>1</samples>
-                <resolution>1.0</resolution>
-                <min_angle>-0.01</min_angle>
-                <max_angle>0.01</max_angle>
-              </horizontal>
-              <vertical>
-                <samples>1</samples>
-                <resolution>1</resolution>
-                <min_angle>-0.01</min_angle>
-                <max_angle>0.01</max_angle>
-              </vertical>
-          </scan>
-          <range>
-              <min>0.01</min>
-              <max>3.75</max>
-              <resolution>0.02</resolution>
-          </range>
-        </ray>
-      <plugin filename="libgazebo_ros_range.so" name="gazebo_ros_range">
-        <gaussianNoise>0.005</gaussianNoise>
-        <updateRate>5</updateRate>
-        <topicName>/tip_sensor/height_above_ground</topicName>
-        <frameName>tip</frameName>
-        <radiation>infrared</radiation>
-        <fov>0.02</fov>
-      </plugin>
-    </sensor>
-  </gazebo>
 </robot>
